File: alim_row.kicad_sch (KiCad schematic)
At the start: 100 parts, among them J631 Conn_01x01, J632 Conn_01x01, J633 Conn_01x01, J634 Conn_01x01, J635 Conn_01x01, J636 Conn_01x01, J637 Conn_01x01, J638 Conn_01x01, J639 Conn_01x01, J640 Conn_01x01, J641 Conn_01x01, J642 Conn_01x01, J643 Conn_01x01, J644 Conn_01x01, J645 Conn_01x01, J646 Conn_01x01, J647 Conn_01x01, J648 Conn_01x01, J649 Conn_01x01, J650 Conn_01x01, J651 Conn_01x01, J652 Conn_01x01, J653 Conn_01x01, J654 Conn_01x01, J655 Conn_01x01, J656 Conn_01x01, J657 Conn_01x01, J658 Conn_01x01, J659 Conn_01x01, J660 Conn_01x01, J661 Conn_01x01, J662 Conn_01x01, J663 Conn_01x01, J664 Conn_01x01, J665 Conn_01x01, J666 Conn_01x01, J667 Conn_01x01, J668 Conn_01x01, J669 Conn_01x01, J670 Conn_01x01, J671 Conn_01x01, J672 Conn_01x01, J673 Conn_01x01, J674 Conn_01x01, J675 Conn_01x01, J676 Conn_01x01, J677 Conn_01x01, J678 Conn_01x01, J679 Conn_01x01, J680 Conn_01x01, J681 Conn_01x01, J682 Conn_01x01, J683 Conn_01x01, J684 Conn_01x01, J685 Conn_01x01, J686 Conn_01x01, J687 Conn_01x01, J688 Conn_01x01, J689 Conn_01x01, J690 Conn_01x01, J691 Conn_01x01, J692 Conn_01x01, J693 Conn_01x01, J694 Conn_01x01, J695 Conn_01x01, J696 Conn_01x01, J697 Conn_01x01, J698 Conn_01x01, J699 Conn_01x01, J700 Conn_01x01, J701 Conn_01x01, J702 Conn_01x01, J703 Conn_01x01, J704 Conn_01x01, J705 Conn_01x01, J706 Conn_01x01, J707 Conn_01x01, J708 Conn_01x01, J709 Conn_01x01, J710 Conn_01x01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

Commit message: [ADD] footprints placed
Connections:
- net at J706.1 (Pin_1), J707.1 (Pin_1), J708.1 (Pin_1)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: no longer J681.1 (Pin_1), J682.1 (Pin_1), J683.1 (Pin_1), J684.1 (Pin_1), J685.1 (Pin_1), J686.1 (Pin_1), J687.1 (Pin_1), J688.1 (Pin_1), J689.1 (Pin_1), J690.1 (Pin_1), J691.1 (Pin_1), J692.1 (Pin_1), J693.1 (Pin_1), J694.1 (Pin_1), J695.1 (Pin_1), J696.1 (Pin_1), J697.1 (Pin_1), J698.1 (Pin_1), J699.1 (Pin_1), J700.1 (Pin_1), J701.1 (Pin_1), J702.1 (Pin_1), J703.1 (Pin_1), J704.1 (Pin_1), J705.1 (Pin_1)
- net at J631.1 (Pin_1), J632.1 (Pin_1), J633.1 (Pin_1)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: no longer J656.1 (Pin_1), J657.1 (Pin_1), J658.1 (Pin_1), J659.1 (Pin_1), J660.1 (Pin_1), J661.1 (Pin_1), J662.1 (Pin_1), J663.1 (Pin_1), J664.1 (Pin_1), J665.1 (Pin_1), J666.1 (Pin_1), J667.1 (Pin_1), J668.1 (Pin_1), J669.1 (Pin_1), J670.1 (Pin_1), J671.1 (Pin_1), J672.1 (Pin_1), J673.1 (Pin_1), J674.1 (Pin_1), J675.1 (Pin_1), J676.1 (Pin_1), J677.1 (Pin_1), J678.1 (Pin_1), J679.1 (Pin_1), J680.1 (Pin_1)
- new net: J656.1 (Pin_1), J657.1 (Pin_1), J658.1 (Pin_1), J659.1 (Pin_1), J660.1 (Pin_1), J661.1 (Pin_1), J662.1 (Pin_1), J663.1 (Pin_1), J664.1 (Pin_1), J665.1 (Pin_1), J666.1 (Pin_1), J667.1 (Pin_1), J668.1 (Pin_1), J669.1 (Pin_1), J670.1 (Pin_1), J671.1 (Pin_1), J672.1 (Pin_1), J673.1 (Pin_1), J674.1 (Pin_1), J675.1 (Pin_1), J676.1 (Pin_1), J677.1 (Pin_1), J678.1 (Pin_1), J679.1 (Pin_1), J680.1 (Pin_1)
- new net: J681.1 (Pin_1), J682.1 (Pin_1), J683.1 (Pin_1), J684.1 (Pin_1), J685.1 (Pin_1), J686.1 (Pin_1), J687.1 (Pin_1), J688.1 (Pin_1), J689.1 (Pin_1), J690.1 (Pin_1), J691.1 (Pin_1), J692.1 (Pin_1), J693.1 (Pin_1), J694.1 (Pin_1), J695.1 (Pin_1), J696.1 (Pin_1), J697.1 (Pin_1), J698.1 (Pin_1), J699.1 (Pin_1), J700.1 (Pin_1), J701.1 (Pin_1), J702.1 (Pin_1), J703.1 (Pin_1), J704.1 (Pin_1), J705.1 (Pin_1)
Changed lines of the file:
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@@
-	)
-	(junction
-		(at 134.62 20.32)
-		(diameter 0)
-		(color 0 0 0 0)
 	)
 	(junction
@@
 	)
 	(junction
-		(at 111.76 20.32)
-		(diameter 0)
-		(color 0 0 0 0)
-	)
-	(junction
 		(at 66.04 58.42)
 		(diameter 0)
@@
 	)
 	(junction
-		(at 111.76 58.42)
-		(diameter 0)
-		(color 0 0 0 0)
-	)
-	(junction
 		(at 43.18 30.48)
 		(diameter 0)
@@
 		(color 0 0 0 0)
 	)
-	(junction
-		(at 134.62 58.42)
-		(diameter 0)
-		(color 0 0 0 0)
-	)
 	(wire
 		(pts
@@
 	(wire
 		(pts
-			(xy 111.76 20.32) (xy 134.62 20.32)
-		)
-		(stroke
-			(width 0)
-			(type default)
-		)
-	)
-	(wire
-		(pts
 			(xy 203.2 25.4) (xy 203.2 30.48)
 		)
@@
 		)
 		(stroke
-			(width 0)
-			(type default)
-		)
-	)
-	(wire
-		(pts
-			(xy 111.76 58.42) (xy 134.62 58.42)
-		)
-		(stroke
